File: CUR_flight_computer_25-26/CUR_flight_computer_25-26.kicad_pcb (KiCad board)
At the start: 2 copper layers, 144 parts, among them J1 3220-14-0100-00, J10 PYRO, J11 PYRO, J12 USB_C_Receptacle_USB2.0_16P, J13 Conn_01x04_Pin, J14 Conn_Coaxial_Small, J2 Screw_Terminal_01x02, J3 Screw_Terminal_01x02, J4 XT30PW-M, J5 XT30PW-M, J6 Micro_SD_Card, J7 Conn_01x02_Pin, J8 PYRO, J9 PYRO, Q1 NTR4003N, SW1 GSPTS0018, SW2 SW_SPDT, SW3 GSPTS0018, SW4 GSPTS0018, SW5 GSPTS0018, U1 STM32H523VETx, U10 W25Q32JVSS, U11 SAM-M8Q, U12 BUK9K25-40RAX, U13 BUK9K25-40RAX, U14 USBLC6-2SC6, U2 IIS2MDC, U3 LPS22HB, U4 LSM6DSV80X, U5 E22-400M30S, U6 BU33SD5, U7 LM66200, U8 ZXCT180A4W5, U9 ZXCT180A4W5, Y1 16M18PX/XT324-10/10

Commit message: Update CUR_flight_computer_25-26.kicad_pcb
Parts:
- moved C26 186.2 mm to (239.7, 135.8)
- moved C27 181.1 mm to (239.2, 129.6)
- moved R9 178.9 mm to (242.9, 126.3)
- moved C25 177.0 mm to (235.0, 123.6)
- moved R8 176.9 mm to (239.2, 126.3)
- moved R7 153.2 mm to (201.8, 136.3)
- moved R54 132.7 mm to (235.9, 67.0)
- moved R55 132.5 mm to (235.9, 68.8)
- moved R56 130.4 mm to (235.1, 63.6)
- moved J13 120.5 mm to (217.1, 70.4), turned to 180 degrees
- moved R52 113.0 mm to (195.8, 103.5)
- moved R53 110.1 mm to (196.1, 100.8)
- moved Q1 109.0 mm to (206.1, 69.9)
- moved R51 107.8 mm to (196.1, 97.7), turned to 180 degrees
- moved R49 106.7 mm to (204.4, 72.2)
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
Commit message: Update CUR_flight_computer_25-26.kicad_pcb
Parts:
- moved C33 219.5 mm to (261.6, 89.1)
- moved R29 219.4 mm to (261.7, 95.9)
- moved R28 219.4 mm to (261.7, 93.6)
- moved C31 210.8 mm to (253.8, 57.2)
- moved C32 210.8 mm to (253.8, 59.7)
- moved C24 192.4 mm to (250.1, 80.9)
- moved C23 192.2 mm to (250.0, 78.7)
- moved R5 190.8 mm to (246.3, 76.1)
- moved C18 184.8 mm to (239.0, 81.8)
- moved C19 184.8 mm to (239.0, 84.3)
- moved R4 179.0 mm to (235.2, 77.9)
- moved R21 177.0 mm to (219.2, 99.7)
- moved R22 176.4 mm to (219.3, 95.7)
- moved C20 175.2 mm to (222.8, 58.3)
- moved C21 175.2 mm to (222.8, 60.8)
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
Commit message: more small organization
Parts:
- moved R6 157.2 mm to (236.0, 38.4), turned to 180 degrees
- moved R1 118.7 mm to (211.5, 48.5)
- moved C17 116.3 mm to (215.5, 68.5), turned to 90 degrees
- moved C16 108.3 mm to (208.7, 85.8), turned to 180 degrees
- moved U8 106.6 mm to (184.0, 101.3), turned to 180 degrees
- moved R2 105.1 mm to (205.3, 85.8)
- moved C1 44.6 mm to (128.7, 102.2)
- moved C2 44.6 mm to (128.7, 104.7)
- moved C3 44.6 mm to (128.7, 107.2)
- moved C4 44.6 mm to (128.7, 109.7)
- moved C5 44.6 mm to (128.7, 112.2)
- moved FB1 44.6 mm to (140.7, 107.2)
- moved C10 44.6 mm to (132.7, 112.2)
- moved C11 44.6 mm to (136.7, 102.2)
- moved C12 44.6 mm to (136.7, 104.7)
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
Commit message: more more organization
Parts:
- moved C1 98.2 mm to (226.8, 97.6), turned to 180 degrees
- moved C8 94.9 mm to (226.7, 94.0), turned to 180 degrees
- moved C13 84.9 mm to (213.7, 71.5)
- moved C11 79.3 mm to (215.3, 91.5), turned to 180 degrees
- moved C14 79.3 mm to (208.7, 76.4), turned to -90 degrees
- moved D15 60.5 mm to (167.8, 81.5)
- moved R44 54.7 mm to (178.4, 83.5)
- moved R45 50.2 mm to (178.4, 81.3), turned to 180 degrees
- moved D16 48.6 mm to (166.1, 67.3)
- moved R39 47.2 mm to (178.4, 79.4), turned to 180 degrees
- moved R37 46.3 mm to (181.2, 74.2), turned to 180 degrees
- moved R31 46.2 mm to (177.8, 74.2)
- moved R36 46.1 mm to (181.3, 71.5)
- moved D14 42.6 mm to (165.9, 54.8)
- moved R32 41.1 mm to (177.9, 71.5)
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Connections:
- R31 pad 2: Net-(U12B-G2) -> Net-(U13A-G1)
- R33 pad 1: Net-(U12B-G2) -> Net-(U13A-G1)
- R38 pad 2: Net-(U13A-G1) -> Net-(U12B-G2)
- R40 pad 1: Net-(U13A-G1) -> Net-(U12B-G2)
- U12 pad 6: Net-(J9-Pin_1) -> Net-(J10-Pin_1)
- U13 pad 5: Net-(J10-Pin_1) -> Net-(J9-Pin_1)

Commit message: ah
Parts:
- moved R16 125.4 mm to (195.1, 111.7), turned to 90 degrees
- moved R14 125.4 mm to (192.7, 117.2)
- moved R15 125.2 mm to (192.7, 118.9), turned to 180 degrees
- moved D5 123.7 mm to (192.5, 124.0)
- moved R17 123.2 mm to (193.3, 111.8), turned to 90 degrees
- moved R18 120.8 mm to (187.1, 117.5), turned to 180 degrees
- moved C29 119.6 mm to (184.0, 112.0), turned to -90 degrees
- moved D10 119.5 mm to (187.2, 105.6), turned to 180 degrees
- moved D7 117.9 mm to (187.6, 123.9), turned to 180 degrees
- moved R13 117.5 mm to (187.2, 103.6)
- moved R11 115.3 mm to (179.7, 116.7)
- moved R12 112.9 mm to (180.0, 103.4), turned to 180 degrees
- moved D4 112.8 mm to (180.2, 123.9)
- moved D9 112.5 mm to (180.0, 105.7)
- moved U9 111.9 mm to (188.2, 111.8), turned to 180 degrees
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
Commit message: most of layout figured out
trouble finding room for power
Parts:
- removed D13: ESDZV5HS-1BF4, Diode_SMD:D_0201_0603Metric
- added D15: ESDZV5HS-1BF4, Diode_SMD:D_0201_0603Metric, F.Cu at (63.1, 51.3)
- added D16: ESDZV5HS-1BF4, Diode_SMD:D_0201_0603Metric, F.Cu at (156.7, 50.8)
- J13: footprint Resistor_SMD:R_0603_1608Metric -> Connector_PinHeader_2.54mm:PinHeader_1x04_P2.54mm_Vertical
- moved J14 206.4 mm to (48.7, 115.5), turned to 0 degrees
- moved R9 205.9 mm to (52.8, 117.3), turned to 90 degrees
- moved C26 203.7 mm to (52.8, 113.6), turned to 90 degrees
- moved C27 200.4 mm to (54.8, 117.5), turned to 90 degrees
- moved R8 183.0 mm to (73.3, 148.5)
- moved C33 180.4 mm to (82.0, 106.2), turned to 90 degrees
- moved C31 175.5 mm to (78.7, 69.0), turned to -90 degrees
- moved C32 173.6 mm to (80.4, 69.0), turned to -90 degrees
- moved C24 172.9 mm to (80.2, 112.8)
- moved J6 172.7 mm to (92.2, 67.0)
- moved R28 172.7 mm to (89.1, 99.7), turned to 90 degrees
- moved C23 172.7 mm to (80.4, 110.8)
- moved U4 172.7 mm to (76.3, 111.8)
- moved R5 171.5 mm to (78.0, 109.0), turned to 180 degrees
- moved C18 170.8 mm to (70.8, 111.4), turned to -90 degrees
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Connections:
- C1 pad 1: +3.3V -> +3V3
- C11 pad 1: +3.3V -> +3V3
- C12 pad 1: +3.3V -> +3V3
- C13 pad 1: +3.3V -> +3V3
- C14 pad 1: +3.3V -> +3V3
- C2 pad 1: +3.3V -> +3V3
- C4 pad 1: +3.3V -> +3V3
- C6 pad 1: +3.3V -> +3V3
- C8 pad 1: +3.3V -> +3V3
- D14 pad 1: Net-(D14-A1) -> GND
- FB1 pad 1: +3.3V -> +3V3
- J10 pad 2: Net-(D16-A1) -> BATT_PYRO
- J11 pad 2: Net-(D15-A1) -> BATT_PYRO
- J8 pad 2: Net-(D13-A1) -> BATT_PYRO
- J9 pad 2: Net-(D14-A1) -> BATT_PYRO
- R3 pad 1: +3.3V -> +3V3
- R4 pad 1: +3.3V -> +3V3
- R5 pad 1: +3.3V -> +3V3
- R7 pad 1: +3.3V -> +3V3
- SW2 pad 3: +3.3V -> +3V3
- U1 pad 100: +3.3V -> +3V3
- U1 pad 11: +3.3V -> +3V3
- U1 pad 28: +3.3V -> +3V3
- U1 pad 50: +3.3V -> +3V3
- U1 pad 6: +3.3V -> +3V3
- U1 pad 73: +3.3V -> +3V3
- U1 pad 75: +3.3V -> +3V3
Routing:
- added copper zone on In2.Cu, net +3V3
- added copper zone on B.Cu, net GND
- added copper zone on F.Cu, net GND
- added copper zone on In1.Cu, net GND
Other:
- board outline added: 54.2 x 110 mm
- copper layers 2 -> 4

Commit message: trying to figure out layout
Parts:
- added D13: ESDZV5HS-1BF4, Diode_SMD:D_0201_0603Metric, F.Cu at (-9.15, 54.5)
- R8: moved to B.Cu
- moved J2 150.6 mm to (65.8, 23.1)
- moved J3 150.6 mm to (78.5, 23.1)
- moved D16 99.9 mm to (57.3, 52.3), turned to 0 degrees
- moved J10 96.9 mm to (51.8, 46.1), turned to -90 degrees
- moved U14 95.2 mm to (143.3, 45.2), turned to 0 degrees
- moved J6 94.0 mm to (18.2, 125.0)
- moved J12 93.9 mm to (152.6, 49.2), turned to 90 degrees
- moved C32 92.9 mm to (7.14, 126.1)
- moved C31 92.9 mm to (5.39, 126.2)
- moved D11 92.9 mm to (7.14, 122.2)
- moved D12 92.9 mm to (7.14, 130.4)
- moved C29 91.9 mm to (121.5, 36.6)
- moved D10 91.9 mm to (124.7, 30.3)
- moved D8 91.9 mm to (107.9, 38.2)
- moved R15 91.9 mm to (130.2, 43.6)
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Other:
- board size 54.2 x 110 mm -> 54.2 x 120 mm

Commit message: semi decent layout
Parts:
- removed the D16 at (57.3, 52.3)
- removed D3, D8: ESDZV5HS-1BF4, Diode_SMD:D_0201_0603Metric
- C11, C18, C19, C20, C21, C22, C23, C24, C30, D17, Q1, R20, R21, R22, R23, R24, R25, R26, R27, R3, R4, R48, R49, R5, U10, U2, U3, U4: moved to B.Cu
- moved SW3 163.9 mm to (78.8, 56.8)
- moved SW4 163.9 mm to (71.6, 56.8)
- moved SW5 163.9 mm to (64.3, 56.8)
- moved LED_2 161.3 mm to (90.8, 127.2), turned to 180 degrees
- moved R56 154.4 mm to (95.6, 129.7), turned to 180 degrees
- moved R54 153.0 mm to (94.8, 126.2), turned to 180 degrees
- moved R55 151.6 mm to (94.8, 124.5), turned to 180 degrees
- moved C9 148.5 mm to (53.2, 88.1), turned to -45 degrees
- moved Y1 142.6 mm to (55.2, 86.0), turned to -135 degrees
- moved C3 136.6 mm to (57.5, 83.8), turned to -45 degrees
- moved R51 107.1 mm to (95.6, 115.7)
- moved R52 107.1 mm to (95.4, 121.5)
- moved R53 107.1 mm to (95.7, 118.8)
- moved LED_1 107.1 mm to (91.0, 118.5)
- moved SW2 92.2 mm to (129.0, 81.8)
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Other:
- board size 54.2 x 120 mm -> 53.2 x 117.5 mm
