File: CUR_flight_computer_25-26/CUR_flight_computer_25-26.kicad_pcb (KiCad board)
At the start: 4 copper layers, 41.5 x 71.4 mm, 187 parts, among them J10 PYRO, J11 PYRO, J12 USB_C_Receptacle_USB2.0_16P, J13 Conn_01x04_Pin, J14 Conn_Coaxial_Small, J15 FTSH-107-01-X-DV-K-TR, J2 Screw_Terminal_01x02, J3 Screw_Terminal_01x02, J4 XT30PW-M, J5 XT30PW-M, J6 Micro_SD_Card, J7 Conn_01x02_Pin, J8 PYRO, J9 PYRO, Q1 NTR4003N, SW1 GSPTS0018, SW2 SW_SPDT, SW3 GSPTS0018, SW4 GSPTS0018, SW5 GSPTS0018, U1 STM32H523VETx, U10 W25Q32JVSS, U11 SAM-M8Q, U12 BUK9K25-40RAX, U13 BUK9K25-40RAX, U14 USBLC6-2SC6, U2 IIS2MDC, U3 LPS22HB, U4 LSM6DSV80X, U5 E22-400MM_22S, U6 BU33SD5, U7 LM66200, U8 ZXCT180A4W5, U9 ZXCT180A4W5, Y1 16M18PX/XT324-10/10

Commit message: more layout yay
Parts:
- C31, C32, TP41: moved to B.Cu
- moved TP41 105.7 mm to (87.9, 88.7), turned to 90 degrees
- moved R48 28.8 mm to (76.3, 98.2), turned to 0 degrees
- moved BZ1 28.2 mm to (81.8, 89.3), turned to 90 degrees
- moved R49 28.1 mm to (76.3, 99.7), turned to 180 degrees
- moved Q1 21.8 mm to (79.8, 99.0), turned to 0 degrees
- moved D17 18.9 mm to (81.5, 95.5), turned to 0 degrees
- moved R34 12.5 mm to (79.5, 64.6), turned to 180 degrees
- moved R35 12.0 mm to (76.4, 64.6), turned to 180 degrees
- moved R36 11.7 mm to (57.1, 73.5), turned to 0 degrees
- moved R20 11.5 mm to (77.5, 65.8)
- moved R37 10.8 mm to (60.2, 73.5)
- moved C32 8.37 mm to (68.6, 89.8), turned to 0 degrees
- moved C30 7.20 mm to (76.2, 75.3), turned to 90 degrees
- moved J10 7.02 mm to (85.0, 73.0)
- moved J8 6.99 mm to (85.0, 66.0)
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Connections:
- BZ1 pad 1: (no net) -> +3V3
- BZ1 pad 2: (no net) -> Net-(D17-A)
- J4 pad 1: GND -> /Power/BATT_SWITCH
- J4 pad 2: /Power/BATT_SWITCH -> GND
- J5 pad 1: GND -> PYRO_BATT_SWITCH
- J5 pad 2: PYRO_BATT_SWITCH -> GND
