File: CUR_flight_computer_25-26/power.kicad_sch (KiCad schematic)
At the start: 28 parts, among them J2 Screw_Terminal_01x02, J3 Screw_Terminal_01x02, J4 XT30PW-M, J5 XT30PW-M, U6 BU33SD5, U7 LM66200, U8 ZXCT180A4W5, U9 ZXCT180A4W5

Commit message: added new header footprint
Parts:
- J2, J3: footprint TerminalBlock_Phoenix:TerminalBlock_Phoenix_PT-1,5-2-5.0-H_1x02_P5.00mm_Horizontal -> Terminal_SAMESKY_TB0011-350-02GR:SAMESKY_TB0011-350-02GR
Changed lines of the file:
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@@
 			)
 		)
-		(property "Footprint" "TerminalBlock_Phoenix:TerminalBlock_Phoenix_PT-1,5-2-5.0-H_1x02_P5.00mm_Horizontal"
+		(property "Footprint" "Terminal_SAMESKY_TB0011-350-02GR:SAMESKY_TB0011-350-02GR"
 			(at 40.64 135.89 0)
 			(effects
@@
 			)
 		)
-		(property "Footprint" "TerminalBlock_Phoenix:TerminalBlock_Phoenix_PT-1,5-2-5.0-H_1x02_P5.00mm_Horizontal"
+		(property "Footprint" "Terminal_SAMESKY_TB0011-350-02GR:SAMESKY_TB0011-350-02GR"
 			(at 40.64 166.37 0)
 			(effects
