File: CUR_flight_computer_25-26/power.kicad_sch (KiCad schematic)
At the start: 26 parts, among them J2 Screw_Terminal_01x02, J3 Screw_Terminal_01x02, J4 XT30U-M, J5 XT30U-M, U6 BU33SD5, U7 LM66200, U8 ZXCT180A4W5, U9 ZXCT180A4W5

Commit message: Begin layout
Parts:
- removed D10, D9: LED, LED_SMD:LED_0603_1608Metric, symbol Device:LED
- removed R12, R13: 150, Resistor_SMD:R_0603_1608Metric, symbol Device:R_Small_US
- removed U8, U9: ZXCT180A4W5, Package_TO_SOT_SMD:SOT-23-5, symbol DI_ZXCT180:ZXCT180A4
- added U15, U16: ZXCT180B4W5, Package_TO_SOT_SMD:SOT-23-5, symbol DI_ZXCT180:ZXCT180B4
- R18: value 5mOhm 1W -> CSSH0805FT1L00; footprint Resistor_SMD:R_1206_3216Metric -> Resistor_SMD:R_0805_2012Metric
- R19: value 1mOhm 1W -> CSSH0805FT1L00; footprint Resistor_SMD:R_2010_5025Metric -> Resistor_SMD:R_0805_2012Metric
Connections:
- net +3V3: now also U15.5 (VS), U16.5 (VS)
- net +BATT: now also U15.3 (IN-)
- net BATT_MEAS: now also J2.2 (Pin_2), U15.1 (IN+); no longer J2.1 (Pin_1)
- net BATT_PYRO: now also U16.3 (IN-)
- net BATT_SWITCH: now also J2.1 (Pin_1); no longer J2.2 (Pin_2)
- net GND: now also U15.2 (GND), U16.2 (GND)
- net I_SENSE: now also U15.4 (OUT)
- net I_SENSE_PYRO: now also U16.4 (OUT)
- net PYRO_BATT_MEAS: now also U16.1 (IN+)
Other:
- note added: "1mOhm 1W"
- note removed: "Indicator LEDs"
- note removed: "PE1206FKM470R005Z - expensive ass resistor"
- note removed: "check LDO and main rail power check if pyro battery connected"
